File: Mainboard.kicad_pcb (KiCad board)
At the start: 4 copper layers, 70 x 60 mm, 213 parts, among them J1 JTAG, J101 USB1, J2 Power, J201 USB1, J4 Expansion, J501 USB1, J601 DAC1, J611 DAC2, J621 DAC3, J701 ADC1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

Commit message: Update to KiCad 6
Parts:
- H1, H2, H3, H4: footprint MountingHole:MountingHole_2.7mm_M2.5_DIN965_Pad -> MountingHole:MountingHole_3.2mm_M3_DIN965_Pad
