File: Mainboard.kicad_sch (KiCad schematic)
At the start: 7 parts

Commit message: Update to KiCad 6
Parts:
- H1, H2, H3, H4: footprint MountingHole:MountingHole_2.7mm_M2.5_DIN965_Pad -> MountingHole:MountingHole_3.2mm_M3_DIN965_Pad
